File: hardware/PCB/RTC Module/RTC_GL/RTC_GL.kicad_pcb (KiCad board)
At the start: 2 copper layers, 44 x 55 mm, 12 parts, among them J1 Screw_Terminal_01x04, U1 DS1307+, X1 32.768KHz

Commit message: Added 3D models to pcb of RTC (real time clock) module.
Parts:
- moved D1 1.00 mm to (99.0, 64.0)
Routing:
- net Net-(D1-A): track 9.12 -> 8.12 mm
- net GND: track 78.9 -> 79.9 mm
Changed lines of the file:
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@@
 			)
 		)
+		(model "${PROJECT_LIB_3D}/MFR1WSFRF52-4K32.STEP"
+			(offset
+				(xyz 10 0 0)
+			)
+			(scale
+				(xyz 1.5 1 1)
+			)
+			(rotate
+				(xyz -90 -0 -0)
+			)
+		)
 	)
 	(footprint "TerminalBlock_Phoenix:TerminalBlock_Phoenix_MPT-0,5-4-2.54_1x04_P2.54mm_Horizontal"
@@
 			)
 		)
+		(model "${PROJECT_LIB_3D}/Screw Terminal Block 3.5mm Blue 4-way.step"
+			(offset
+				(xyz 4 0 0)
+			)
+			(scale
+				(xyz 0.8 0.8 0.8)
+			)
+			(rotate
+				(xyz -90 -0 -0)
+			)
+		)
 	)
 	(footprint "LED_THT:LED_D3.0mm"
 		(layer "F.Cu")
-		(at 99.02 63 180)
+		(at 99.02 64 180)
 		(descr "LED, diameter 3.0mm, 2 pins, generated by kicad-footprint-generator")
 		(tags "LED")
@@
 			)
 		)
+		(model "${PROJECT_LIB_3D}/LED_WP7113SRD_E.STEP"
+			(offset
+				(xyz 1.25 0 0)
+			)
+			(scale
+				(xyz 1 1 1)
+			)
+			(rotate
+				(xyz -90 -0 -0)
+			)
+		)
 	)
 	(footprint "Package_DIP:DIP-8_W7.62mm"
@@
 			)
 		)
+		(model "/home/farzad/Desktop/GreenLink/hardware/PCB/lib/3D models/DS1307+.STEP"
+			(offset
+				(xyz 4 -3.75 0.5)
+			)
+			(scale
+				(xyz 1 1 1)
+			)
+			(rotate
+				(xyz -90 -0 -0)
+			)
+		)
 	)
 	(footprint "Diode_THT:D_DO-41_SOD81_P10.16mm_Horizontal"
@@
 			)
 		)
+		(model "/home/farzad/Desktop/GreenLink/hardware/PCB/lib/3D models/1N4933-T.STEP"
+			(offset
+				(xyz 5 0 0)
+			)
+			(scale
+				(xyz 1 1 1)
+			)
+			(rotate
+				(xyz -90 -0 -0)
+			)
+		)
 	)
 	(footprint "Crystal:Crystal_C38-LF_D3.0mm_L8.0mm_Horizontal"
@@
 			)
 		)
+		(model "/home/farzad/Desktop/GreenLink/hardware/PCB/lib/3D models/DS26-L3N-32.768KHZ-8.2PF-20PPM-TW.STEP"
+			(offset
+				(xyz 1 0 3)
+			)
+			(scale
+				(xyz 1 1 1)
+			)
+			(rotate
+				(xyz -90 -0 -0)
+			)
+		)
 	)
 	(footprint "LED_THT:LED_D3.0mm"
@@
 			)
 		)
+		(model "${PROJECT_LIB_3D}/LED_WP7113SRD_E.STEP"
+			(offset
+				(xyz 1.5 0 0)
+			)
+			(scale
+				(xyz 1 1 1)
+			)
+			(rotate
+				(xyz -90 -0 -0)
+			)
+		)
 	)
 	(footprint "Capacitor_THT:C_Disc_D6.0mm_W2.5mm_P5.00mm"
@@
 			)
 		)
+		(model "${PROJECT_LIB_3D}/FG24X7R1A106KRT00--3DModel-STEP-269445.STEP"
+			(offset
+				(xyz 2.5 0 0)
+			)
+			(scale
+				(xyz 1 1 1)
+			)
+			(rotate
+				(xyz -90 -0 -0)
+			)
+		)
 	)
 	(footprint "Resistor_THT:R_Axial_DIN0309_L9.0mm_D3.2mm_P20.32mm_Horizontal"
@@
 			)
 		)
+		(model "${PROJECT_LIB_3D}/MFR1WSFRF52-4K32.STEP"
+			(offset
+				(xyz 10.5 0 0)
+			)
+			(scale
+				(xyz 1.5 1 1)
+			)
+			(rotate
+				(xyz -90 -0 -0)
+			)
+		)
 	)
 	(footprint "Battery:BatteryHolder_MYOUNG_BS-07-A1BJ001_CR2032"
@@
 			)
 		)
+		(model "/home/farzad/Desktop/GreenLink/hardware/PCB/lib/3D models/KLS5-CR2032-01 battery holder.stp"
+			(offset
+				(xyz 12.5 0 0)
+			)
+			(scale
+				(xyz 1 1 1)
+			)
+			(rotate
+				(xyz -0 -0 -0)
+			)
+		)
 	)
 	(footprint "Resistor_THT:R_Axial_DIN0309_L9.0mm_D3.2mm_P20.32mm_Horizontal"
@@
 			)
 		)
+		(model "${PROJECT_LIB_3D}/MFR1WSFRF52-4K32.STEP"
+			(offset
+				(xyz 10 0 0)
+			)
+			(scale
+				(xyz 1.5 1 1)
+			)
+			(rotate
+				(xyz -90 -0 -0)
+			)
+		)
 	)
 	(footprint "Resistor_THT:R_Axial_DIN0309_L9.0mm_D3.2mm_P20.32mm_Horizontal"
@@
 			)
 		)
+		(model "${PROJECT_LIB_3D}/MFR1WSFRF52-4K32.STEP"
+			(offset
+				(xyz 10 0 0)
+			)
+			(scale
+				(xyz 1.5 1 1)
+			)
+			(rotate
+				(xyz -90 -0 -0)
+			)
+		)
 	)
 	(gr_rect
@@
 	)
 	(segment
-		(start 96.48 64.89)
-		(end 96.48 63)
+		(start 101.59 70)
+		(end 96.48 64.89)
 		(width 0.7)
 		(layer "B.Cu")
@@
 	)
 	(segment
-		(start 101.59 70)
-		(end 96.48 64.89)
+		(start 96.48 64.89)
+		(end 96.48 64)
 		(width 0.7)
 		(layer "B.Cu")
@@
 	)
 	(segment
-		(start 99.02 63)
-		(end 99.02 57.75)
+		(start 99.02 57.75)
+		(end 99.02 64)
 		(width 0.7)
 		(layer "B.Cu")
