File: hardware/PCB/Motor Channel Module/MC_GL/MC_GL.kicad_sch (KiCad schematic)
At the start: 8 parts, among them J2 S_T_01x02, J5 Screw_Terminal_01x06, Q1 NPN, U1 12v

Commit message: Designed Motor Channel module and also added it's 3D components
Parts:
- added D1, D5: LED, LED_THT:LED_D5.0mm, symbol Device:LED
- added D3, D6: 1N4002, Diode_THT:D_DO-41_SOD81_P10.16mm_Horizontal, symbol Diode:1N4002
- added J1, J3: S_T_01x02, TerminalBlock:TerminalBlock_MaiXu_MX126-5.0-02P_1x02_P5.00mm, symbol Connector:Screw_Terminal_01x02
- added J4, J6, J7, J8: Screw_Terminal_01x03, TerminalBlock:TerminalBlock_MaiXu_MX126-5.0-03P_1x03_P5.00mm, symbol Connector:Screw_Terminal_01x03
- added Q2, Q3: NPN, Transistors_BJT:2N2222, symbol Simulation_SPICE:NPN
- added R3, R5: 4.7K, Resistor_THT:R_Axial_DIN0309_L9.0mm_D3.2mm_P20.32mm_Horizontal, symbol Device:R
- added R4, R6: 1K, Resistor_THT:R_Axial_DIN0309_L9.0mm_D3.2mm_P20.32mm_Horizontal, symbol Device:R
- added U2, U3: 12v, Relays:HJR-3FF-S-Z, symbol HJR-3FF-S-Z:12vDC-Relay
- D2: footprint (none) -> LED_THT:LED_D5.0mm
- J2: footprint (none) -> TerminalBlock:TerminalBlock_MaiXu_MX126-5.0-02P_1x02_P5.00mm
- J5: footprint (none) -> TerminalBlock:TerminalBlock_MaiXu_MX126-5.0-06P_1x06_P5.00mm
- Q1: footprint (none) -> Transistors_BJT:2N2222
- R1, R2: footprint (none) -> Resistor_THT:R_Axial_DIN0309_L9.0mm_D3.2mm_P20.32mm_Horizontal
Connections:
- net 12v: now also J4.2 (Pin_2), J6.2 (Pin_2), J7.2 (Pin_2), J8.2 (Pin_2), U2.1 (SRC), U3.1 (SRC)
- net 5v: now also J4.3 (Pin_3), J6.3 (Pin_3), J7.3 (Pin_3), J8.3 (Pin_3), U2.2 (T1), U3.2 (T1)
- net GND: now also D1.1 (K), D3.2 (A), D5.1 (K), D6.2 (A), J1.2 (Pin_2), J3.2 (Pin_2), J4.1 (Pin_1), J6.1 (Pin_1), J7.1 (Pin_1), J8.1 (Pin_1), Q2.3 (E), Q3.3 (E)
- net IN2: now also R3.1, R4.1
- net IN3: now also R5.1, R6.1
- new net: D1.2 (A), R3.2
- new net: D5.2 (A), R5.2
- new net: D3.1 (K), J1.1 (Pin_1), U2.4 (OC)
- new net: D6.1 (K), J3.1 (Pin_1), U3.4 (OC)
- new net: Q3.1 (C), U3.3 (T2)
- new net: Q2.2 (B), R4.2
- new net: Q2.1 (C), U2.3 (T2)
- new net: Q3.2 (B), R6.2
Other:
- note added: "Channel 2"
- note added: "Channel 3"
